File: PCB#1/PCB#1.kicad_pcb (KiCad board)
At the start: 2 copper layers, 2 parts

Commit message: Add files via upload
Parts:
- removed REF**: QFN-56-1EP_7x7mm_P0.4mm_EP3.2x3.2mm, Package_DFN_QFN:QFN-56-1EP_7x7mm_P0.4mm_EP3.2x3.2mm
- removed REF**: InvenSense_QFN-24_3x3mm_P0.4mm, Sensor_Motion:InvenSense_QFN-24_3x3mm_P0.4mm
Routing:
- net (no net): track 88.5 -> 0.00 mm

Commit message: Add files via upload
Parts:
- added C1: 10uF, Capacitor_SMD:C_0603_1608Metric, F.Cu at (153.8, 118.5)
- added C10: 100nF, Capacitor_SMD:C_0603_1608Metric, F.Cu at (151.2, 104.5)
- added C11: 1uF, Capacitor_SMD:C_0603_1608Metric, F.Cu at (154.5, 114.0)
- added C12: 100nF, Capacitor_SMD:C_0603_1608Metric, F.Cu at (150.5, 116.0)
- added C13: 100nF, Capacitor_SMD:C_0603_1608Metric, F.Cu at (147.0, 116.0)
- added C14: 100nF, Capacitor_SMD:C_0603_1608Metric, F.Cu at (159.5, 109.0)
- added C15: 100nF, Capacitor_SMD:C_0603_1608Metric, F.Cu at (158.0, 109.0)
- added C16: 1uF, Capacitor_SMD:C_0603_1608Metric, F.Cu at (153.3, 100.3)
- added C17: 100nF, Capacitor_SMD:C_0603_1608Metric, F.Cu at (141.0, 110.5)
- added C18: 1uF, Capacitor_SMD:C_0603_1608Metric, F.Cu at (151.8, 100.3)
- added C19: 10uF, Capacitor_SMD:C_0603_1608Metric, F.Cu at (128.0, 104.2)
- added C2: 15pF, Capacitor_SMD:C_0603_1608Metric, F.Cu at (143.0, 105.5)
- added C20: 100nF, Capacitor_SMD:C_0603_1608Metric, F.Cu at (127.2, 106.5)
- added C21: 100nF, Capacitor_SMD:C_0603_1608Metric, F.Cu at (130.2, 112.8)
- added C22: 10uF, Capacitor_SMD:C_0603_1608Metric, F.Cu at (128.0, 102.0)
- added C23: 100nF, Capacitor_SMD:C_0603_1608Metric, F.Cu at (127.2, 109.5)
- added C24: 100nF, Capacitor_SMD:C_0603_1608Metric, F.Cu at (154.5, 115.5)
- added C3: 15pF, Capacitor_SMD:C_0603_1608Metric, F.Cu at (140.2, 103.0)
- added C4: 10uF, Capacitor_SMD:C_0603_1608Metric, F.Cu at (155.2, 118.5)
- added C5: 100nF, Capacitor_SMD:C_0603_1608Metric, F.Cu at (164.5, 98.5)
- added C6: 100nF, Capacitor_SMD:C_0603_1608Metric, F.Cu at (156.5, 109.0)
- added C7: 100nF, Capacitor_SMD:C_0603_1608Metric, F.Cu at (141.0, 112.0)
- added C8: 1uF, Capacitor_SMD:C_0603_1608Metric, F.Cu at (154.5, 112.5)
- added C9: 100nF, Capacitor_SMD:C_0603_1608Metric, F.Cu at (147.2, 104.5)
- added J2: Conn_01x02, Connector_PinHeader_2.54mm:PinHeader_1x02_P2.54mm_Vertical, F.Cu at (163.8, 102.0)
- added P1: USB_C_Plug_USB2.0, Connector_USB:USB_C_Receptacle_HRO_TYPE-C-31-M-12, F.Cu at (170.8, 109.2)
- added Q1: BSS138, Package_TO_SOT_SMD:SOT-23, F.Cu at (129.8, 115.6)
- added R1: 27.4, Resistor_SMD:R_0603_1608Metric, F.Cu at (161.9, 109.9)
- added R13: 4.7k, Resistor_SMD:R_0603_1608Metric, F.Cu at (137.2, 117.0)
- added R14: 4.7k, Resistor_SMD:R_0603_1608Metric, F.Cu at (135.2, 117.0)
- added R15: 4.7k, Resistor_SMD:R_0603_1608Metric, F.Cu at (134.8, 107.8)
- added R16: 4.7k, Resistor_SMD:R_0603_1608Metric, F.Cu at (134.8, 109.5)
- added R2: 27.4, Resistor_SMD:R_0603_1608Metric, F.Cu at (161.9, 108.4)
- added R3: 1k, Resistor_SMD:R_0603_1608Metric, F.Cu at (162.8, 98.5)
- added R4: 1k, Resistor_SMD:R_0603_1608Metric, F.Cu at (141.0, 109.0)
- added R5: 5.1k, Resistor_SMD:R_0603_1608Metric, F.Cu at (164.7, 111.1)
- added R6: 27.4, Resistor_SMD:R_0603_1608Metric, F.Cu at (157.2, 113.2)
- added R7: 4.7k, Resistor_SMD:R_0603_1608Metric, F.Cu at (130.2, 106.8)
- added R8: 4.7k, Resistor_SMD:R_0603_1608Metric, F.Cu at (132.2, 115.5)
- added R9: 4.7k, Resistor_SMD:R_0603_1608Metric, F.Cu at (127.2, 112.5)
- added U1: RP2040, Package_DFN_QFN:QFN-56-1EP_7x7mm_P0.4mm_EP3.2x3.2mm, F.Cu at (148.0, 110.2)
- added U2: ICM-20948, Sensor_Motion:InvenSense_QFN-24_3x3mm_P0.4mm, F.Cu at (130.2, 109.8)
- added U3: NCP1117-3.3_SOT223, Package_TO_SOT_SMD:SOT-223-3_TabPin2, F.Cu at (161.8, 117.0)
- added U4: W25Q128JVS, Package_SO:SOIC-8_5.3x5.3mm_P1.27mm, F.Cu at (159.0, 101.8)
- added U5: NCP1117-1.8_SOT223, Package_TO_SOT_SMD:SOT-223-3_TabPin2, F.Cu at (134.0, 102.0)
- added U7: MPL115A1, Package_LGA:NXP_LGA-8_3x5mm_P1.25mm_H1.2mm, F.Cu at (149.0, 100.3)
- added U8: TCA9406DC, Package_SO:VSSOP-8_3x3mm_P0.65mm, F.Cu at (136.2, 113.8)
- added Y1: Crystal_GND24, Crystal:Crystal_SMD_Abracon_ABM8G-4Pin_3.2x2.5mm, F.Cu at (140.2, 106.0)
Routing:
- net GND: track 0.00 -> 198.8 mm, vias 0 -> 12
- net +3V3: track 0.00 -> 176.1 mm, vias 0 -> 2
- net +1V1: track 0.00 -> 62.3 mm, vias 0 -> 4
- net +1V8: track 0.00 -> 56.8 mm
- net /QSPI_SD1: track 0.00 -> 42.5 mm
- net /QSPI_SD2: track 0.00 -> 40.2 mm
- net VBUS: track 0.00 -> 30.7 mm
- net /QSPI_SD0: track 0.00 -> 21.7 mm
- net /QSPI_SCLK: track 0.00 -> 20.4 mm
- net /QSPI_SD3: track 0.00 -> 19.1 mm
- net /GPIO18: track 0.00 -> 19.0 mm
- net /GPIO17: track 0.00 -> 16.1 mm
- net Net-(U1-USB_DM): track 0.00 -> 13.1 mm
- net /GPIO13: track 0.00 -> 12.0 mm
- net /GPIO16: track 0.00 -> 10.9 mm
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